File: Main.brd (EAGLE design)
At the start: 160 x 100 mm, 18 parts, among them X1 736880-49, X2 736880-49

Commit message: [rm]いったん全部消去
Parts:
- removed C1, C2, C3, C4, C5, C6: (no value), capacitor-wima:C10B5
- removed R1, R2, R3, R4, R5, R6: (no value), rcl:0207/5V
- removed TR1, TR2: 166L8, trafo-hammondmfg:C8H
- removed V1, V2: (no value), VacuumTube:NOVAL
- removed X1, X2: 736880-49, con-conrad:736880-49
Connections:
- removed net GND: C2.2, C4.2, C5.2, C6.2, R1.1, R2.1, R3.1, R5.1
- removed net N$1: C2.1, R5.2, V2.3
- removed net N$12: C1.1, X2.2
- removed net N$2: C6.1, R6.2, V2.9
- removed net N$3: C3.2, R2.2, V1.2
- removed net N$4: C1.2, R1.2, V2.2
- removed net N$5: TR2.BLK@1, V1.7
- removed net N$6: TR1.BLK@1, V2.7
- removed net N$7: C3.1, X1.2
- removed net N$8: C4.1, R3.2, V1.3
- removed net N$9: C5.1, R4.2, V1.9
- removed net VCC: R4.1, R6.1, TR1.BLK@2, TR2.BLK@2

Commit message: [add]全回路作成
Parts:
- added C1, C2, C3, C6, C7, C8: 0.1u, VacuumTube:C025-025X050
- added C10, C5: 10u, VacuumTube:C025-025X050
- added C4, C9: 170, VacuumTube:C025-025X050
- added JP1, JP2, JP3, JP4, JP5, JP6: (no value), VacuumTube:1X02
- added R1, R10, R16, R7: 220k, VacuumTube:0207/7
- added R11, R2: 3.83k, VacuumTube:0207/7
- added R12, R3: 50k, VacuumTube:0207/7
- added R13, R4: 1M, VacuumTube:0207/7
- added R14, R5: 1.5k, VacuumTube:0207/7
- added R15, R6: 100k, VacuumTube:0207/7
- added R17, R8: 220u, VacuumTube:0207/7
- added R18, R9: 2k, VacuumTube:0207/7
- added V1, V2, V3, V4: (no value), VacuumTube:AT-MT9P
Connections:
- new net GND: C10.2, C4.2, C5.2, C9.2, JP1.1, JP2.1, JP3.1, JP4.1, R1.1, R10.1, R11.1, R15.1, R16.2, R17.2, R2.1, R6.1, R7.2, R8.2, V1.9, V2.18, V3.9, V4.18
- new net N$1: R3.1, V1.7
- new net N$10: C2.1
- new net N$11: V1.18, V3.18
- new net N$12: C3.1
- new net N$13: C3.2, R7.1, V2.14
- new net N$14: C4.1, R8.1, V2.16
- new net N$15: V2.5
- new net N$16: JP5.1
- new net N$17: C5.1, R9.1, V2.1
- new net N$18: JP6.1
- new net N$19: R12.1, V3.7
- new net N$2: R2.2, V1.3
- new net N$20: R11.2, V3.3
- new net N$21: C6.2, R10.2, V3.5
- new net N$22: C6.1
- new net N$23: R14.2, V3.16
- new net N$24: R13.1, R14.1, R15.2
- new net N$25: C7.2, R13.2, V3.14
- new net N$26: C7.1
- new net N$27: C8.1
- new net N$28: C8.2, R16.1, V4.14
- new net N$29: C9.1, R17.1, V4.16
- new net N$3: JP2.2
- new net N$30: V4.5
- new net N$31: C10.1, R18.1, V4.1
- new net N$4: JP1.2
- new net N$5: C1.2, R1.2, V1.5
- new net N$6: R5.2, V1.16
- new net N$7: C1.1
- new net N$8: R4.1, R5.1, R6.2
- new net N$9: C2.2, R4.2, V1.14
- new net VCC: JP3.2, JP5.2, JP6.2, R12.2, R18.2, R3.2, R9.2, V1.12, V3.12
- new net VCC/2: JP4.2, V1.1, V2.9, V3.1, V4.9

Commit message: [fix]ピンのラベルを編集
Parts:
- removed JP2, JP3, JP5, JP6: (no value), VacuumTube:1X02
- added INPUT2, OUT_TRANSFORMER1, OUT_TRANSFORMER2, VCC: (no value), VacuumTube:1X02
- moved C10 165.8 mm to (83.8, -179.1)
- moved C3 165.8 mm to (77.5, -64.8)
- moved C9 165.8 mm to (77.5, -179.1)
- moved R10 165.8 mm to (91.4, -179.1)
- moved R11 165.8 mm to (101.6, -179.1)
- moved R12 165.8 mm to (111.8, -179.1)
- moved R13 165.8 mm to (121.9, -179.1)
- moved C1 165.8 mm to (77.5, 19.1)
- moved C2 165.8 mm to (77.5, 14.0)
- moved C4 165.8 mm to (77.5, -69.8)
- moved C5 165.8 mm to (77.5, -85.1)
- moved R1 165.8 mm to (78.7, 49.5)
- moved R15 165.8 mm to (88.9, -186.7)
- moved R2 165.8 mm to (78.7, 44.5)
- moved R3 165.8 mm to (78.7, 39.4)
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- renumbered JP1 to INPUT1, JP4 to HEATER_VCC
Connections:
- net GND: now also INPUT2.1, VCC.1; no longer JP2.1, JP3.1
- net N$16: now also OUT_TRANSFORMER1.1; no longer JP5.1
- net N$18: now also OUT_TRANSFORMER2.1; no longer JP6.1
- net N$3: now also INPUT2.2; no longer JP2.2
- net VCC: now also OUT_TRANSFORMER1.2, OUT_TRANSFORMER2.2, VCC.2; no longer JP3.2, JP5.2, JP6.2

Commit message: [fix]基板に絶望している
Parts:
- moved OUT_TRANSFORMER1 266.6 mm to (-146.0, 55.1)
- moved R9 255.4 mm to (-115.8, 70.2)
- moved C3 255.1 mm to (-114.5, 103.2)
- moved C4 255.1 mm to (-114.5, 98.2)
- moved C5 255.1 mm to (-114.5, 82.9)
- moved R7 255.1 mm to (-113.3, 93.1)
- moved R8 255.1 mm to (-113.3, 88.0)
- moved V4 237.5 mm to (47.0, 61.9), turned to 90 degrees
- moved R1 206.9 mm to (-126.5, 23.2)
- moved C10 204.7 mm to (44.8, 21.9)
- moved C9 204.7 mm to (38.5, 21.9)
- moved R10 204.7 mm to (52.4, 21.9)
- moved R11 204.7 mm to (62.6, 21.9)
- moved R12 204.7 mm to (72.8, 21.9)
- moved R13 204.7 mm to (82.9, 21.9)
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Connections:
- net GND: now also V1.4, V2.5, V3.4, V4.5; no longer V1.9, V2.18, V3.9, V4.18
- net N$1: now also V1.6; no longer V1.7
- net N$11: now also V1.5, V3.5; no longer V1.18, V3.18
- net N$13: now also V2.2; no longer V2.14
- net N$14: now also V2.3; no longer V2.16
- net N$15: now also V2.7; no longer V2.5
- net N$17: now also V2.9; no longer V2.1
- net N$19: now also V3.6; no longer V3.7
- net N$2: now also V1.8; no longer V1.3
- net N$20: now also V3.8; no longer V3.3
- net N$21: now also V3.7; no longer V3.5
- net N$23: now also V3.3; no longer V3.16
- net N$25: now also V3.2; no longer V3.14
- net N$28: now also V4.2; no longer V4.14
- net N$29: now also V4.3; no longer V4.16
- net N$30: now also V4.7; no longer V4.5
- net N$31: now also V4.9; no longer V4.1
- net N$5: now also V1.7; no longer V1.5
- net N$6: now also V1.3; no longer V1.16
- net N$9: now also V1.2; no longer V1.14
- net VCC: now also V1.1, V3.1; no longer V1.12, V3.12
- net VCC/2: now also V1.9, V2.4, V3.9, V4.4; no longer V1.1, V2.9, V3.1, V4.9
Routing:
- net N$32: track 0.00 -> 114.0 mm
Other:
- board size 160 x 100 mm -> 310 x 114 mm

Commit message: [fix]重大な欠陥を直した
Parts:
- C9: value 170 -> 220u
- R17: value 220u -> 170
Changed lines of the file:
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@@
 <attribute name="VALUE" x="132.254" y="53.966" size="1.27" layer="27" ratio="10"/>
 </element>
-<element name="C9" library="VacuumTube" library_urn="urn:adsk.eagle:library:8044196" package="C025-025X050" package3d_urn="urn:adsk.eagle:package:8969349/1" value="170" x="38.47" y="21.93" smashed="yes">
+<element name="C9" library="VacuumTube" library_urn="urn:adsk.eagle:library:8044196" package="C025-025X050" package3d_urn="urn:adsk.eagle:package:8969349/1" value="220u" x="38.47" y="21.93" smashed="yes">
 <attribute name="NAME" x="36.184" y="23.454" size="1.27" layer="25" ratio="10"/>
 <attribute name="VALUE" x="36.184" y="19.136" size="1.27" layer="27" ratio="10"/>
@@
 <attribute name="VALUE" x="57.774" y="13.7512" size="1.27" layer="27" ratio="10"/>
 </element>
-<element name="R17" library="VacuumTube" library_urn="urn:adsk.eagle:library:8044196" package="0207/7" package3d_urn="urn:adsk.eagle:package:8969348/1" value="220u" x="70.22" y="14.31" smashed="yes">
+<element name="R17" library="VacuumTube" library_urn="urn:adsk.eagle:library:8044196" package="0207/7" package3d_urn="urn:adsk.eagle:package:8969348/1" value="170" x="70.22" y="14.31" smashed="yes">
 <attribute name="NAME" x="67.68" y="15.707" size="1.27" layer="25" ratio="10"/>
 <attribute name="VALUE" x="67.934" y="13.7512" size="1.27" layer="27" ratio="10"/>

Commit message: [fix]重大な欠陥
Parts:
- C4: value 170 -> 220u
- R8: value 220u -> 170
Changed lines of the file:
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@@
 <attribute name="VALUE" x="-116.816" y="100.436" size="1.27" layer="27" ratio="10"/>
 </element>
-<element name="C4" library="VacuumTube" library_urn="urn:adsk.eagle:library:8044196" package="C025-025X050" package3d_urn="urn:adsk.eagle:package:8969349/1" value="170" x="-114.53" y="98.15" smashed="yes">
+<element name="C4" library="VacuumTube" library_urn="urn:adsk.eagle:library:8044196" package="C025-025X050" package3d_urn="urn:adsk.eagle:package:8969349/1" value="220u" x="-114.53" y="98.15" smashed="yes">
 <attribute name="NAME" x="-116.816" y="99.674" size="1.27" layer="25" ratio="10"/>
 <attribute name="VALUE" x="-116.816" y="95.356" size="1.27" layer="27" ratio="10"/>
@@
 <attribute name="VALUE" x="-115.546" y="92.5112" size="1.27" layer="27" ratio="10"/>
 </element>
-<element name="R8" library="VacuumTube" library_urn="urn:adsk.eagle:library:8044196" package="0207/7" package3d_urn="urn:adsk.eagle:package:8969348/1" value="220u" x="-113.26" y="87.99" smashed="yes">
+<element name="R8" library="VacuumTube" library_urn="urn:adsk.eagle:library:8044196" package="0207/7" package3d_urn="urn:adsk.eagle:package:8969348/1" value="170" x="-113.26" y="87.99" smashed="yes">
 <attribute name="NAME" x="-115.8" y="89.387" size="1.27" layer="25" ratio="10"/>
 <attribute name="VALUE" x="-115.546" y="87.4312" size="1.27" layer="27" ratio="10"/>

Commit message: [fix]手直し
Connections:
- net GND: now also V1.9, V3.9; no longer V1.4, V3.4
- net VCC/2: now also V1.4, V3.4; no longer V1.9, V3.9
Changed lines of the file:
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@@
 <contactref element="R6" pad="1"/>
 <contactref element="R1" pad="1"/>
-<contactref element="V1" pad="4"/>
+<contactref element="V1" pad="9"/>
 <contactref element="V2" pad="5"/>
 <contactref element="R7" pad="2"/>
@@
 <contactref element="R8" pad="2"/>
 <contactref element="C5" pad="2"/>
-<contactref element="V3" pad="4"/>
+<contactref element="V3" pad="9"/>
 <contactref element="R11" pad="1"/>
 <contactref element="R10" pad="1"/>
@@
 <wire x1="-113.26" y1="98.15" x2="-109.45" y2="93.07" width="0" layer="19" extent="1-1"/>
 <wire x1="-47.51" y1="71.07" x2="-109.45" y2="93.07" width="0" layer="19" extent="1-1"/>
-<wire x1="145.61" y1="40.2" x2="-113.26" y2="82.91" width="0" layer="19" extent="1-1"/>
-<wire x1="-72.75" y1="34.24" x2="-47.51" y2="71.07" width="0" layer="19" extent="1-1"/>
-<wire x1="-66.77" y1="35.91" x2="-72.75" y2="34.24" width="0" layer="19" extent="1-1"/>
+<wire x1="117.51" y1="40.2" x2="-113.26" y2="82.91" width="0" layer="19" extent="1-1"/>
+<wire x1="-100.85" y1="34.24" x2="-47.51" y2="71.07" width="0" layer="19" extent="1-1"/>
+<wire x1="-66.77" y1="35.91" x2="-100.85" y2="34.24" width="0" layer="19" extent="1-1"/>
 <wire x1="-120.11" y1="28.29" x2="-66.77" y2="35.91" width="0" layer="19" extent="1-1"/>
 <wire x1="-130.27" y1="23.21" x2="-120.11" y2="28.29" width="0" layer="19" extent="1-1"/>
@@
 <wire x1="-147.57" y1="23.49" x2="-147.92" y2="15.06" width="0" layer="19" extent="1-1"/>
 <wire x1="-147.206" y1="32.9774" x2="-147.57" y2="23.49" width="0" layer="19" extent="1-1"/>
-<wire x1="15.95" y1="70.73" x2="145.61" y2="40.2" width="0" layer="19" extent="1-1"/>
+<wire x1="15.95" y1="70.73" x2="117.51" y2="40.2" width="0" layer="19" extent="1-1"/>
 <wire x1="58.79" y1="21.93" x2="15.95" y2="70.73" width="0" layer="19" extent="1-1"/>
 <wire x1="63.87" y1="14.31" x2="58.79" y2="21.93" width="0" layer="19" extent="1-1"/>
@@
 <signal name="VCC/2">
 <contactref element="HEATER_VCC" pad="2"/>
-<contactref element="V1" pad="9"/>
+<contactref element="V1" pad="4"/>
 <contactref element="V2" pad="4"/>
-<contactref element="V3" pad="9"/>
+<contactref element="V3" pad="4"/>
 <contactref element="V4" pad="4"/>
-<wire x1="44.05" y1="91.05" x2="117.51" y2="40.2" width="0" layer="19" extent="1-1"/>
-<wire x1="-19.41" y1="91.39" x2="117.51" y2="40.2" width="0" layer="19" extent="1-1"/>
-<wire x1="-100.85" y1="34.24" x2="-19.41" y2="91.39" width="0" layer="19" extent="1-1"/>
-<wire x1="-145.92" y1="5.58" x2="-100.85" y2="34.24" width="0" layer="19" extent="1-1"/>
+<wire x1="44.05" y1="91.05" x2="145.61" y2="40.2" width="0" layer="19" extent="1-1"/>
+<wire x1="-19.41" y1="91.39" x2="145.61" y2="40.2" width="0" layer="19" extent="1-1"/>
+<wire x1="-72.75" y1="34.24" x2="-19.41" y2="91.39" width="0" layer="19" extent="1-1"/>
+<wire x1="-145.92" y1="5.58" x2="-72.75" y2="34.24" width="0" layer="19" extent="1-1"/>
 </signal>
 <signal name="N$1">

Commit message: [fix]スクリーングリッドの抵抗値と容量を変化
Parts:
- C10, C5: value 10u -> 22u
Changed lines of the file:
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@@
 <attribute name="VALUE" x="-115.546" y="87.4312" size="1.27" layer="27" ratio="10"/>
 </element>
-<element name="C5" library="VacuumTube" library_urn="urn:adsk.eagle:library:8044196" package="C025-025X050" package3d_urn="urn:adsk.eagle:package:8969349/1" value="10u" x="-114.53" y="82.91" smashed="yes">
+<element name="C5" library="VacuumTube" library_urn="urn:adsk.eagle:library:8044196" package="C025-025X050" package3d_urn="urn:adsk.eagle:package:8969349/1" value="22u" x="-114.53" y="82.91" smashed="yes">
 <attribute name="NAME" x="-116.816" y="84.434" size="1.27" layer="25" ratio="10"/>
 <attribute name="VALUE" x="-116.816" y="80.116" size="1.27" layer="27" ratio="10"/>
@@
 <attribute name="VALUE" x="67.934" y="13.7512" size="1.27" layer="27" ratio="10"/>
 </element>
-<element name="C10" library="VacuumTube" library_urn="urn:adsk.eagle:library:8044196" package="C025-025X050" package3d_urn="urn:adsk.eagle:package:8969349/1" value="10u" x="44.82" y="21.93" smashed="yes">
+<element name="C10" library="VacuumTube" library_urn="urn:adsk.eagle:library:8044196" package="C025-025X050" package3d_urn="urn:adsk.eagle:package:8969349/1" value="22u" x="44.82" y="21.93" smashed="yes">
 <attribute name="NAME" x="42.534" y="23.454" size="1.27" layer="25" ratio="10"/>
 <attribute name="VALUE" x="42.534" y="19.136" size="1.27" layer="27" ratio="10"/>
