File: Main.brd (EAGLE design)
At the start: 310 x 114 mm, 38 parts

Commit message: [fix]直し
Parts:
- removed C10: 22u, VacuumTube:C025-025X050
- removed C9: 220u, VacuumTube:C025-025X050
- removed R18, R9: 2k, VacuumTube:0207/7
- C4: device VacuumTube:C025-025X050 -> VacuumTube:E2,5-6
- C5: value 22u -> 220u; device VacuumTube:C025-025X050 -> VacuumTube:E2,5-6
- R11, R2: value 3.83k -> 3.9k
- R12, R3: value 50k -> 51k
- R17, R8: value 170 -> 180
- moved C4 109.1 mm to (-149.9, -5.08)
- moved C5 101.9 mm to (-149.9, -12.7)
Connections:
- removed net N$11: V1.5, V3.5
- removed net VCC/2: HEATER_VCC.2, V1.4, V2.4, V3.4, V4.4
- net GND: now also C4.-, C5.-; no longer C10.2, C4.2, C5.2, C9.2
- net N$14: now also C4.+; no longer C4.1
- net N$17: no longer C5.1, R9.1
- net N$29: now also C5.+; no longer C9.1
- net N$31: no longer C10.1, R18.1
- net VCC: now also HEATER_VCC.2, V1.4, V1.5, V2.4, V3.4, V3.5, V4.4; no longer R18.2, R9.2
