File: Main_LEFT.sch (EAGLE design)
At the start: 34 parts

Commit message: [fix]右と左分けた
Parts:
- removed C5: 220u, VacuumTube:CAPACITOR2
- removed C6, C7, C8: 0.1u, VacuumTube:C
- removed INPUT1, INPUT2, OUT_TRANSFORMER1, OUT_TRANSFORMER2: (no value), VacuumTube:PINHD-1X2
- removed R10, R16: 220k, VacuumTube:RESISTOR2
- removed R11: 3.9k, VacuumTube:RESISTOR2
- removed R12: 51k, VacuumTube:RESISTOR2
- removed R13: 1M, VacuumTube:RESISTOR2
- removed R14: 1.5k, VacuumTube:RESISTOR2
- removed R15: 100k, VacuumTube:RESISTOR2
- removed R17: 180, VacuumTube:RESISTOR2
- removed V3: (no value), VacuumTube:AT-MT9P(12AX7)
- removed V4: (no value), VacuumTube:AT-MT9P(6BQ5)
- added INPUT, OUT_TRANSFORMER: (no value), VacuumTube:PINHD-1X2
Connections:
- removed net N$18: OUT_TRANSFORMER2.1
- removed net N$19: R12.1, V3A.TA
- removed net N$20: R11.2, V3A.TK
- removed net N$21: C6.2, R10.2, V3A.TG
- removed net N$22: C6.1
- removed net N$23: R14.2, V3B.TK
- removed net N$24: R13.1, R14.1, R15.2
- removed net N$25: C7.2, R13.2, V3B.TG
- removed net N$26: C7.1
- removed net N$27: C8.1
- removed net N$28: C8.2, R16.1, V4A.PG
- removed net N$29: C5.+, R17.1, V4A.PK
- removed net N$3: INPUT2.2
- removed net N$30: V4A.PA
- removed net N$31: V4A.PSG
- net GND: now also INPUT.1; no longer C5.-, INPUT1.1, INPUT2.1, R10.1, R11.1, R15.1, R16.2, R17.2, V3C.H2, V4B.H2
- net N$16: now also OUT_TRANSFORMER.1; no longer OUT_TRANSFORMER1.1
- net N$4: now also INPUT.2; no longer INPUT1.2
- net VCC: now also OUT_TRANSFORMER.2; no longer OUT_TRANSFORMER1.2, OUT_TRANSFORMER2.2, R12.2, V3B.TA, V3C.H1, V3C.H3, V4B.H1
Other:
- note added: "FIRST_OUT"
- note added: "INPUT"
- note added: "SECOND_OUT"
- note added: "THIRD_OUT"
- note removed: "FIRST_OUT1"
- note removed: "FIRST_OUT2"
- note removed: "INPUT1"
- note removed: "INPUT2"
- note removed: "SECOND_OUT1"
- note removed: "SECOND_OUT2"
- note removed: "THIRD_OUT1"
- note removed: "THIRD_OUT2"
- moved on the sheet: C1, C2, C3, C4, R1, R2, R3, R4, R5, R6, R7, R8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
