File: Main_RIGHT.brd (EAGLE design)
At the start: 155 x 114 mm, 18 parts

Commit message: [fix]ボード作成
Parts:
- moved C2 230.1 mm to (-115.0, 26.6)
- moved R4 229.5 mm to (-114.7, 21.8)
- moved R5 229.2 mm to (-114.6, 31.8)
- moved R6 228.8 mm to (-114.4, 36.8)
- moved V1 220.1 mm to (-91.1, 8.20)
- moved OUT_TRANSFORMER 216.7 mm to (-108.4, 93.5)
- moved HEATER_VCC 162.8 mm to (-81.4, 93.5)
- moved C1 144.8 mm to (-72.4, 30.6)
- moved R1 144.4 mm to (-72.2, 25.8)
- moved R2 144.1 mm to (-72.1, 20.8)
- moved R3 143.8 mm to (-71.9, 35.8)
- moved VCC 136.8 mm to (-68.4, 93.5)
- moved R7 106.4 mm to (-53.2, 78.9)
- moved R8 106.1 mm to (-53.1, 95.9)
- moved C3 105.4 mm to (-52.7, 84.6)
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